File: Grogu Badge/Electronics/Grogu.kicad_sch (KiCad schematic)
At the start: 75 parts, among them J1 TYPE-C-31-M-12, J3 S3B-PH-SM4-TB(LF)(SN), SW1 BOOT, SW2 ENABLE, U1 USBLC6-2SC6, U2 SPX3819M5-L-3-3, U3 W25Q128JVSIQ, U4 ESP32-C3, U5 NS4150, U6 SN74LVC2T45DCUR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

Commit message: new mac
Parts:
- removed AE1: SWRA117D-Left, !Library:SWRA117D_2.4GHz_Left, symbol !Library:SWRA117D-Left
- removed C1, C10, C12, C13, C16, C17, C2, C29, C3, C30, C31, C32, C33, C4, C5, C8: 100n, Capacitor_SMD:C_0402_1005Metric, symbol Device:C
- removed C11, C14: 3p3, Capacitor_SMD:C_0402_1005Metric, symbol Device:C
- removed C15, C20: 10p, Capacitor_SMD:C_0402_1005Metric, symbol Device:C
- removed C18, C19, C25, C6, C7, C9: 10u, Capacitor_SMD:C_0603_1608Metric, symbol Device:C
- removed C21: 4.7n, Capacitor_SMD:C_0402_1005Metric, symbol Device:C
- removed C22: 220u, Capacitor_SMD:CP_Elec_6.3x7.7, symbol Device:C
- removed C23, C27: 1u, Capacitor_SMD:C_0805_2012Metric, symbol Device:C
- removed C24: 2.2n, Capacitor_SMD:C_0402_1005Metric, symbol Device:C
- removed C26: 1n, Capacitor_SMD:C_0402_1005Metric, symbol Device:C
- removed C28: 22p, Capacitor_SMD:C_0402_1005Metric, symbol Device:C
- removed D1: LED, LED_SMD:LED_0805_2012Metric, symbol Device:LED
- removed D10, D4, D5, D6, D7, D8, D9: SK6803MINI-E, LED_SMD:LED_SK6812MINI_PLCC4_3.5x3.5mm_P1.75mm, symbol LED:WS2812B
- removed D13, D14: LESD5D5.0CT1G, Diode_SMD:D_SOD-523, symbol Device:D_TVS
- removed J1: TYPE-C-31-M-12, Connector_USB:USB_C_Receptacle_HRO_TYPE-C-31-M-12, symbol Connector:USB_C_Receptacle_USB2.0
- removed J3: S3B-PH-SM4-TB(LF)(SN), Connector_JST:JST_PH_S3B-PH-SM4-TB_1x03-1MP_P2.00mm_Horizontal, symbol Connector:Conn_01x03_Male
- removed L2, L3: 2n2, Inductor_SMD:L_0402_1005Metric, symbol Device:L
- removed LS1: Speaker, !Library:Speaker-0.5W-8Ohm, symbol Device:Speaker
- removed MK1: ICS-43434, !Library:ICS-43434, symbol !Library:ICS-43434
- removed R1, R4: 5k1, Resistor_SMD:R_0402_1005Metric, symbol Device:R
- removed R10, R13, R9: 1K, Resistor_SMD:R_0402_1005Metric, symbol Device:R
- removed R11: 10K, Resistor_SMD:R_0402_1005Metric, symbol Device:R
- removed R12: 100K, Resistor_SMD:R_0402_1005Metric, symbol Device:R
- removed R14, R15: 30K, Resistor_SMD:R_0402_1005Metric, symbol Device:R
- removed SW1: BOOT, !Library:TS-1187A-B-A-B, symbol Switch:SW_Push
- removed SW2: ENABLE, !Library:TS-1187A-B-A-B, symbol Switch:SW_Push
- removed TP1, TP2: TestPoint, TestPoint:TestPoint_Pad_1.5x1.5mm, symbol Connector:TestPoint
- removed U1: USBLC6-2SC6, Package_TO_SOT_SMD:SOT-23-6, symbol Power_Protection:USBLC6-2SC6
- removed U2: SPX3819M5-L-3-3, Package_TO_SOT_SMD:SOT-23-5, symbol Regulator_Linear:SPX3819M5-L-3-3
- removed U3: W25Q128JVSIQ, Package_SO:SOIC-8_5.275x5.275mm_P1.27mm, symbol !Library:W25Q128JVSIQ
- removed U4: ESP32-C3, Package_DFN_QFN:QFN-32-1EP_5x5mm_P0.5mm_EP3.45x3.45mm, symbol !Library:ESP32-C3
- removed U5: NS4150, Package_SO:MSOP-8_3x3mm_P0.65mm, symbol !Library:NS4150
- removed U6: SN74LVC2T45DCUR, Package_SO:VSSOP-8_2.4x2.1mm_P0.5mm, symbol Logic_LevelTranslator:SN74LVC2T45DCUR
- removed Y1: 40MHz, Crystal:Crystal_SMD_2520-4Pin_2.5x2.0mm, symbol Device:Crystal_GND24
- added C1, C10, C11, C12, C13: 0.1uF, symbol Device:C_Small
- added C14, C7, C9: 1uF, symbol Device:C_Small
- added C5: 10nF, symbol Device:C_Small
- added C8: 10uF, symbol Device:C_Small
- added R6, R7: 0, symbol Device:R
- added U1: ESP32-S3R8, Package_DFN_QFN:QFN-56-1EP_7x7mm_P0.4mm_EP4x4mm, symbol MCU_Espressif:ESP32-S3
- added U2: W25Q128JVSIQ, Package_SO:SOIC-8_5.23x5.23mm_P1.27mm, symbol Memory_Flash:W25Q128JVS
- L1: value 2n2 -> 2nH; footprint Inductor_SMD:L_0402_1005Metric -> (none); PART# C412264 -> (none); SUPPLIER LCSC -> (none)
- R2, R3: value 5k1 -> 0; footprint Resistor_SMD:R_0402_1005Metric -> (none); PART# C105873 -> (none); SUPPLIER LCSC -> (none)
- R5: value 1K -> 0; footprint Resistor_SMD:R_0402_1005Metric -> (none); PART# C25744 -> (none); SUPPLIER LCSC -> (none)
- R8: value 22R -> 100K; footprint Resistor_SMD:R_0402_1005Metric -> (none); PART# C25092 -> (none); SUPPLIER LCSC -> (none)
Connections:
- net GND: now also C1.2, C10.2, C11.2, C12.2, C13.2, C14.2, C5.2, C7.2, C8.2, C9.2, U1.57 (GND), U2.4 (GND); no longer R3.2, R5.2
- net +3V3 renamed SPIHD
- net SPIHD: now also U2.7 (IO3)
- net +5V renamed VDD3P3
- net VDD3P3: now also C11.1, U1.2 (VDD3P3), U1.3 (VDD3P3)
- net 3V3LED: no longer names the net of R5.1
- net 3V3LED: now also U1.33 (SPICLK)
- net CC1: no longer names the net of R3.1
- net CC1: now also U1.31 (SPIWP)
- net ENABLE: no longer names the net of R2.1
- net ENABLE: now also U1.30 (SPIHD)
- net VBUS renamed VDD33
- net VDD33: now also C1.1, C10.1, C12.1, C5.1, C7.1, C8.1, C9.1, U1.20 (VDD3P3_RTC), U1.46 (VDD3P3_CPU), U1.55 (VDDA), U1.56 (VDDA)
- net XTAL renamed SPICS0
- net SPICS0: now also U1.32 (SPICS0), U2.1 (~{CS})
- net XTAL_P renamed VDD_SPI
- net VDD_SPI: now also C13.1, C14.1, U1.29 (VDD_SPI), U2.8 (VCC)
- new net: R6.1, U1.34 (SPIQ)
- new net: R7.1, U1.35 (SPID)
- new net SPICLK: R5.2, U2.6 (CLK)
- new net SPID: R7.2, U2.5 (DI(IO0))
- new net SPIQ: R6.2, U2.2 (DO(IO1))
- new net SPIWP: R3.2, U2.3 (IO2)
- no-connect marks 10 -> 5
Other:
- note added: "FLASH 0 MB PSRAM 8 MB In-package PSRAM GPIO 33, 34, 35, 36, 37"
- note added: "Flash 3V3 16MB"
- note removed: "(LC - 4) * 2 = C (pF)"
- note removed: "CHECK AMOUNT OF LED WHILE ROUTING AND MAKE CUSTOM FOOTPRINT FOR UPSIDE DOWN"
- note removed: "CHECK DIRECTION WHILE ROUTING"
- note removed: "LNA Z=(35+j10)R ANT Z=50R"
- note removed: "LR to GND left channel"
- note removed: "Need footprint for speaker connector"
- note removed: "TBD (both need to be equal) 100K in LyraT reference design 30K in NS4150 reference design"
- title: Grogu Board -> Grogu Badge
